Commit message: new commit

File: install/mobile_robot/share/mobile_robot/model/robot.xacro (robot description, xacro)
@@ -1 +1,186 @@
-/home/adharsh/Desktop/Swarm-robot/build/mobile_robot/model/robot.xacro
+<?xml version="1.0"?>
+<robot name="differential_drive_robot" xmlns:xacro="http://www.ros.org/wiki/xacro">
+  <!-- Constants -->
+  <xacro:property name="pi_const" value="3.14159265"/>
+  <xacro:property name="r" value="0.15"/> <!-- 5 cm -->
+  <xacro:property name="d" value="0.1"/> <!-- 30 cm between wheels -->
+  <xacro:property name="a" value="1.0"/>
+  <xacro:property name="c" value="0.6"/>
+  <xacro:property name="b" value="0.3"/>
+  <xacro:property name="s1" value="${b/2+r}"/>
+  <xacro:property name="s2" value="${2*r}"/>
+  <xacro:property name="s3" value="${2*r}"/>
+  <xacro:property name="s4" value="${c/2+d/2}"/>
+  <!-- Mass and Inertia-->
+  <xacro:property name="d1" value="2710.0"/>
+  <xacro:property name="d2" value="2710.0"/>
+  <xacro:property name="d3" value="2710.0"/>
+  <xacro:property name="m1" value="${d1*a*b*c}"/>
+  <xacro:property name="m2" value="${d2*pi_const*r*r*d}"/>
+  <xacro:property name="m3" value="${d3*(4.0/3.0)*pi_const*r*r*r}"/>
+  <xacro:property name="Ix_body" value="${(1/12)*m1*(b*b+c*c)}"/>
+  <xacro:property name="Iy_body" value="${(1/12)*m1*(a*a+b*b)}"/>
+  <xacro:property name="Iz_body" value="${(1/12)*m1*(a*a+c*c)}"/>
+  <xacro:property name="Iz_wheel" value="${0.5*m2*r*r}"/>
+  <xacro:property name="I_wheel" value="${(1.0/12.0)*m2*(3.0*r*r+d*d)}"/>
+  <xacro:property name="I_caster" value="${(2.0/5.0)*m3*r*r}"/>
+  <!-- Macros -->
+  <xacro:macro name="inertia_body">
+    <inertial>
+      <origin rpy="0 0 0" xyz="0 0 ${s1}"/>
+      <mass value="${m1}"/>
+      <inertia ixx="${Ix_body}" ixy="0.0" ixz="0.0" iyy="${Iy_body}" iyz="0" izz="${Iz_body}" />
+    </inertial>
+  </xacro:macro>
+  <xacro:macro name="inertia_wheel">
+    <inertial>
+      <origin rpy="1.570795 0 0" xyz="0 0 0"/>
+      <mass value="${m2}"/>
+      <inertia ixx="${I_wheel}" ixy="0.0" ixz="0.0" iyy="${I_wheel}" iyz="0" izz="${Iz_wheel}" />
+    </inertial>
+  </xacro:macro>
+  <xacro:macro name="inertia_caster">
+    <inertial>
+      <origin rpy="0 0 0" xyz="0 0 0"/>
+      <mass value="${m3}"/>
+      <inertia ixx="${I_caster}" ixy="0.0" ixz="0.0" iyy="${I_caster}" iyz="0" izz="${I_caster}" />
+    </inertial>
+  </xacro:macro>
+  <!-- Include additional files -->
+  <xacro:include filename="$(find mobile_robot)/model/robot.gazebo"/>
+  <!-- Base link -->
+  <link name="base_footprint"/>
+  <joint name="body_link_joint" type="fixed">
+    <parent link="base_footprint"/>
+    <child link="body_link"/>
+  </joint>
+  <!-- Body link -->
+  <link name="body_link">
+    <visual>
+      <geometry>
+        <box size="${a} ${c} ${b}"/>
+      </geometry>
+      <origin rpy="0 0 0" xyz="0 0 ${s1}"/>
+    </visual>
+    <collision>
+      <geometry>
+        <box size="${a} ${c} ${b}"/>
+      </geometry>
+      <origin rpy="0 0 0" xyz="0 0 ${s1}"/>
+    </collision>
+    <xacro:inertia_body />
+  </link>
+  <!-- Back right wheel -->
+  <joint name="wheel1_joint" type="continuous">
+    <parent link="body_link"/>
+    <child link="wheel1_link"/>
+    <origin xyz="${-s2} ${-s4} ${r}" rpy="0 0 0"/>
+    <axis xyz="0 1 0"/>
+    <limit effort="50000" velocity="10"/>
+    <dynamics damping="1.0" friction="1.0"/>
+  </joint>
+  <link name="wheel1_link">
+    <visual>
+      <origin rpy="1.570795 0 0" xyz="0 0 0"/>
+      <geometry>
+        <cylinder length="${d}" radius="${r}"/>
+      </geometry>
+    </visual>
+    <collision>
+      <origin rpy="1.570795 0 0" xyz="0 0 0"/>
+      <geometry>
+        <cylinder length="${d}" radius="${r}"/>
+      </geometry>
+    </collision>
+    <xacro:inertia_wheel />
+  </link>
+  <!-- Back left wheel -->
+  <joint name="wheel2_joint" type="continuous">
+    <parent link="body_link"/>
+    <child link="wheel2_link"/>
+    <origin xyz="${-s2} ${s4} ${r}" rpy="0 0 0"/>
+    <axis xyz="0 1 0"/>
+    <limit effort="50000" velocity="10"/>
+    <dynamics damping="1.0" friction="1.0"/>
+  </joint>
+  <link name="wheel2_link">
+    <visual>
+      <origin rpy="1.570795 0 0" xyz="0 0 0"/>
+      <geometry>
+        <cylinder length="${d}" radius="${r}"/>
+      </geometry>
+    </visual>
+    <collision>
+      <origin rpy="1.570795 0 0" xyz="0 0 0"/>
+      <geometry>
+        <cylinder length="${d}" radius="${r}"/>
+      </geometry>
+    </collision>
+    <xacro:inertia_wheel />
+  </link>
+  <!-- Caster wheel -->
+  <joint name="caster_joint" type="fixed">
+    <parent link="body_link"/>
+    <child link="caster_link"/>
+    <origin xyz="${s3} 0 ${r}" rpy="0 0 0"/>
+  </joint>
+  <link name="caster_link">
+    <visual>
+      <origin rpy="0 0 0" xyz="0 0 0"/>
+      <geometry>
+        <sphere radius="${r}"/>
+      </geometry>
+    </visual>
+    <collision>
+      <origin rpy="0 0 0" xyz="0 0 0"/>
+      <geometry>
+        <sphere radius="${r}"/>
+      </geometry>
+    </collision>
+    <xacro:inertia_caster />
+  </link>
+  <!-- Sloped front (wedge) -->
+<joint name="slope_joint" type="fixed">
+  <parent link="body_link"/>
+  <child link="slope_link"/>
+</joint>
+<link name="slope_link">
+  <visual>
+    <origin xyz="${a/2} 0 ${b/2}" rpy="3.14 2.54 0"/> <!-- tilt the wedge -->
+    <geometry>
+      <box size="0.05 ${c} 0.25"/> <!-- thin in X, full width Y, height Z -->
+    </geometry>
+  </visual>
+  <collision>
+    <geometry>
+      <box size="0.05 ${c} 0.25"/>
+    </geometry>
+    <origin xyz="${a/2} 0 ${b/2}" rpy="3.14 2.54 0"/>
+  </collision>
+</link>
+  <!-- Lidar -->
+  <joint name="lidar_joint" type="fixed">
+    <origin xyz="0.0 0 ${b+r}" rpy="0 0 0"/>
+    <parent link="body_link"/>
+    <child link="lidar_link"/>
+  </joint>
+  <link name="lidar_link">
+    <visual>
+      <origin rpy="0 0 0.05" xyz="0 0 0"/>
+      <geometry>
+        <cylinder length="0.1" radius="0.1"/>
+      </geometry>
+    </visual>
+    <collision>
+      <origin rpy="0 0 0" xyz="0 0 0.05"/>
+      <geometry>
+        <cylinder length="0.1" radius="0.1"/>
+      </geometry>
+    </collision>
+    <inertial>
+      <mass value="1e-6"/>
+      <origin rpy="0 0 0" xyz="0 0 0"/>
+      <inertia ixx="1e-6" ixy="0" ixz="0" iyy="1e-6" iyz="0" izz="1e-6"/>
+    </inertial>
+  </link>
+</robot>

File: src/mobile_robot/model/robot.xacro (robot description, xacro)
@@ -159,26 +159,4 @@
   </collision>
 </link>
-<!-- Roller -->
-<!-- <joint name="roller_joint" type="continuous">
-  <parent link="body_link"/>
-  <child link="roller_link"/>
-  <origin xyz="${a} 0 ${s1}" rpy="2.54 0 0"/>
-  <axis xyz="0 0 1"/>
-  <!----rotation axis -->
-  <limit effort="10" velocity="5"/>
-</joint>
-<link name="roller_link">
-<visual>
-<origin xyz="${a/2} 0 ${b/2 + 0.05}" rpy="0 1.5708 0"/>
-  <geometry>
-    <cylinder radius="0.05" length="${c}"/> <!-- length same as body width -->
-  </geometry>
-</visual>
-<collision>
-  <geometry>
-    <cylinder radius="0.05" length="${c}"/>
-  </geometry> <origin xyz="${a/2} 0 0.05" rpy="0 1.5708 0"/>
- </collision>
-</link> -->
   <!-- Lidar -->
   <joint name="lidar_joint" type="fixed">
