Commit message: corrected robot structure

File: install/mobile_robot/share/mobile_robot/model/robot_macro.xacro (robot description, xacro)
@@ -26,5 +26,5 @@
   <xacro:macro name="inertia_body">
     <inertial>
-      <origin rpy="0 0 0" xyz="0 0 ${s1}"/>
+      <origin rpy="0 0 0" xyz="0 0 0"/>
       <mass value="${m1}"/>
       <inertia ixx="${Ix_body}" ixy="0.0" ixz="0.0" iyy="${Iy_body}" iyz="0" izz="${Iz_body}" />
@@ -50,13 +50,14 @@
     <parent link="${robot_name}/base_footprint"/>
     <child link="${robot_name}/body_link"/>
+    <origin xyz="0 0 ${2*r}" rpy="0 0 0"/>
   </joint>
   <link name="${robot_name}/body_link">
     <visual>
         <geometry><box size="${a} ${c} ${b}"/></geometry>
-        <origin rpy="0 0 0" xyz="0 0 ${s1}"/>
+        <origin rpy="0 0 0" xyz="0 0 0"/>
     </visual>
     <collision>
         <geometry><box size="${a} ${c} ${b}"/></geometry>
-        <origin rpy="0 0 0" xyz="0 0 ${s1}"/>
+        <origin rpy="0 0 0" xyz="0 0 0"/>
     </collision>
     <xacro:inertia_body />
@@ -65,5 +66,5 @@
     <parent link="${robot_name}/body_link"/>
     <child link="${robot_name}/wheel1_link"/>
-    <origin xyz="${-s2} ${-s4} ${r}" rpy="0 0 0"/>
+    <origin xyz="${-s2} ${-s4} ${-r}" rpy="0 0 0"/>
     <axis xyz="0 1 0"/>
     <limit effort="5000" velocity="10"/>
@@ -81,8 +82,16 @@
     <xacro:inertia_wheel />
   </link>
+  <gazebo reference="${robot_name}/wheel1_link">
+    <mu1>1.0</mu1>
+    <mu2>1.0</mu2>
+    <kp>1000000.0</kp>
+    <kd>100.0</kd>
+    <minDepth>0.001</minDepth>
+    <maxVel>1.0</maxVel>
+  </gazebo>
   <joint name="${robot_name}/wheel2_joint" type="continuous">
     <parent link="${robot_name}/body_link"/>
     <child link="${robot_name}/wheel2_link"/>
-    <origin xyz="${-s2} ${s4} ${r}" rpy="0 0 0"/>
+    <origin xyz="${-s2} ${s4} ${-r}" rpy="0 0 0"/>
     <axis xyz="0 1 0"/>
     <limit effort="5000" velocity="10"/>
@@ -100,8 +109,17 @@
     <xacro:inertia_wheel />
   </link>
-  <joint name="${robot_name}/caster_joint" type="fixed">
+  <gazebo reference="${robot_name}/wheel2_link">
+    <mu1>1.0</mu1>
+    <mu2>1.0</mu2>
+    <kp>1000000.0</kp>
+    <kd>100.0</kd>
+    <minDepth>0.001</minDepth>
+    <maxVel>1.0</maxVel>
+  </gazebo>
+  <joint name="${robot_name}/caster_joint" type="continuous">
     <parent link="${robot_name}/body_link"/>
     <child link="${robot_name}/caster_link"/>
-    <origin xyz="${s3} 0 ${r}" rpy="0 0 0"/>
+    <origin xyz="${s3} 0 ${-r}" rpy="0 0 0"/>
+    <axis xyz="0 1 0"/>
   </joint>
   <link name="${robot_name}/caster_link">
@@ -116,4 +134,9 @@
     <xacro:inertia_caster />
   </link>
+  <gazebo reference="${robot_name}/caster_link">
+    <mu1>0.0</mu1>
+    <mu2>0.0</mu2>
+    <material>Gazebo/Red</material>
+  </gazebo>
   <joint name="${robot_name}/slope_joint" type="fixed">
     <parent link="${robot_name}/body_link"/>
@@ -122,5 +145,5 @@
   <link name="${robot_name}/slope_link">
     <visual>
-      <origin xyz="${a/2} 0 ${b/2}" rpy="3.14 2.54 0"/>
+      <origin xyz="${a/2} 0 ${-b/2}" rpy="3.14 2.54 0"/>
       <geometry><box size="0.05 ${c} 0.25"/></geometry>
     </visual>
@@ -130,6 +153,10 @@
     </collision>
   </link>
+  <gazebo reference="${robot_name}/slope_link">
+    <mu1>0.0</mu1>
+    <mu2>0.0</mu2>
+  </gazebo>
   <joint name="${robot_name}/lidar_joint" type="fixed">
-    <origin xyz="0.0 0 ${b+r}" rpy="0 0 0"/>
+    <origin xyz="0 0 0" rpy="0 0 0"/>
     <parent link="${robot_name}/body_link"/>
     <child link="${robot_name}/lidar_link"/>
@@ -137,9 +164,9 @@
   <link name="${robot_name}/lidar_link">
     <visual>
-      <origin rpy="0 0 0.05" xyz="0 0 0"/>
+      <origin rpy="0 0 0.05" xyz="0.0 0 ${b/2 + 0.05}"/>
       <geometry><cylinder length="0.1" radius="0.1"/></geometry>
     </visual>
     <collision>
-      <origin rpy="0 0 0" xyz="0 0 0.05"/>
+      <origin rpy="0 0 0" xyz="0.0 0 ${b/2 + 0.05}"/>
       <geometry><cylinder length="0.1" radius="0.1"/></geometry>
     </collision>

Commit message: s shaped with error

File: install/mobile_robot/share/mobile_robot/model/robot_macro.xacro (robot description, xacro)
@@ -12,7 +12,7 @@
   <xacro:property name="s3" value="${2*r}"/>
   <xacro:property name="s4" value="${c/2+d/2}"/>
-  <xacro:property name="d1" value="100.0"/>
-  <xacro:property name="d2" value="100.0"/>
-  <xacro:property name="d3" value="100.0"/>
+  <xacro:property name="d1" value="10.0"/>
+  <xacro:property name="d2" value="10.0"/>
+  <xacro:property name="d3" value="10.0"/>
   <xacro:property name="m1" value="${d1*a*b*c}"/>
   <xacro:property name="m2" value="${d2*pi_const*r*r*d}"/>
