Commit message: bug

File: install/mobile_robot/share/mobile_robot/model/robot1.xacro (robot description, xacro)
@@ -1,5 +1 @@
-<?xml version="1.0"?>
-<robot name="differential_drive_robot" xmlns:xacro="http://www.ros.org/wiki/xacro">
-  <xacro:include filename="$(find mobile_robot)/model/robot_macro.xacro"/>
-  <xacro:differential_drive_robot robot_name="robot1"/>
-</robot>
+/home/adharsh/Desktop/Swarm-robot/build/mobile_robot/model/robot1.xacro

File: install/mobile_robot/share/mobile_robot/model/robot2.xacro (robot description, xacro)
@@ -1,5 +1 @@
-<?xml version="1.0"?>
-<robot name="differential_drive_robot" xmlns:xacro="http://www.ros.org/wiki/xacro">
-  <xacro:include filename="$(find mobile_robot)/model/robot_macro.xacro"/>
-  <xacro:differential_drive_robot robot_name="robot2"/>
-</robot>
+/home/adharsh/Desktop/Swarm-robot/build/mobile_robot/model/robot2.xacro

File: install/mobile_robot/share/mobile_robot/model/robot_macro.xacro (robot description, xacro)
@@ -1,187 +1 @@
-<?xml version="1.0"?>
-<robot xmlns:xacro="http://www.ros.org/wiki/xacro">
-<xacro:macro name="differential_drive_robot" params="robot_name">
-  <xacro:property name="pi_const" value="3.14159265"/>
-  <xacro:property name="r" value="0.15"/>
-  <xacro:property name="d" value="0.1"/>
-  <xacro:property name="a" value="1.0"/>
-  <xacro:property name="c" value="0.6"/>
-  <xacro:property name="b" value="0.3"/>
-  <xacro:property name="s1" value="${b/2+r}"/>
-  <xacro:property name="s2" value="${2*r}"/>
-  <xacro:property name="s3" value="${2*r}"/>
-  <xacro:property name="s4" value="${c/2+d/2}"/>
-  <xacro:property name="d1" value="10.0"/>
-  <xacro:property name="d2" value="10.0"/>
-  <xacro:property name="d3" value="10.0"/>
-  <xacro:property name="m1" value="${d1*a*b*c}"/>
-  <xacro:property name="m2" value="${d2*pi_const*r*r*d}"/>
-  <xacro:property name="m3" value="${d3*(4.0/3.0)*pi_const*r*r*r}"/>
-  <xacro:property name="Ix_body" value="${(1/12)*m1*(b*b+c*c)}"/>
-  <xacro:property name="Iy_body" value="${(1/12)*m1*(a*a+b*b)}"/>
-  <xacro:property name="Iz_body" value="${(1/12)*m1*(a*a+c*c)}"/>
-  <xacro:property name="Iz_wheel" value="${0.5*m2*r*r}"/>
-  <xacro:property name="I_wheel" value="${(1.0/12.0)*m2*(3.0*r*r+d*d)}"/>
-  <xacro:property name="I_caster" value="${(2.0/5.0)*m3*r*r}"/>
-  <xacro:macro name="inertia_body">
-    <inertial>
-      <origin rpy="0 0 0" xyz="0 0 0"/>
-      <mass value="${m1}"/>
-      <inertia ixx="${Ix_body}" ixy="0.0" ixz="0.0" iyy="${Iy_body}" iyz="0" izz="${Iz_body}" />
-    </inertial>
-  </xacro:macro>
-  <xacro:macro name="inertia_wheel">
-    <inertial>
-      <origin rpy="1.570795 0 0" xyz="0 0 0"/>
-      <mass value="${m2}"/>
-      <inertia ixx="${I_wheel}" ixy="0.0" ixz="0.0" iyy="${I_wheel}" iyz="0" izz="${Iz_wheel}" />
-    </inertial>
-  </xacro:macro>
-  <xacro:macro name="inertia_caster">
-    <inertial>
-      <origin rpy="0 0 0" xyz="0 0 0"/>
-      <mass value="${m3}"/>
-      <inertia ixx="${I_caster}" ixy="0.0" ixz="0.0" iyy="${I_caster}" iyz="0" izz="${I_caster}" />
-    </inertial>
-  </xacro:macro>
-  <xacro:include filename="$(find mobile_robot)/model/robot.gazebo"/>
-  <link name="${robot_name}/base_footprint"/>
-  <joint name="${robot_name}/body_link_joint" type="fixed">
-    <parent link="${robot_name}/base_footprint"/>
-    <child link="${robot_name}/body_link"/>
-    <origin xyz="0 0 ${2*r}" rpy="0 0 0"/>
-  </joint>
-  <link name="${robot_name}/body_link">
-    <visual>
-        <geometry><box size="${a} ${c} ${b}"/></geometry>
-        <origin rpy="0 0 0" xyz="0 0 0"/>
-    </visual>
-    <collision>
-        <geometry><box size="${a} ${c} ${b}"/></geometry>
-        <origin rpy="0 0 0" xyz="0 0 0"/>
-    </collision>
-    <xacro:inertia_body />
-  </link>
-  <joint name="${robot_name}/wheel1_joint" type="continuous">
-    <parent link="${robot_name}/body_link"/>
-    <child link="${robot_name}/wheel1_link"/>
-    <origin xyz="${-s2} ${-s4} ${-r}" rpy="0 0 0"/>
-    <axis xyz="0 1 0"/>
-    <limit effort="5000" velocity="10"/>
-    <dynamics damping="1.0" friction="1.0"/>
-  </joint>
-  <link name="${robot_name}/wheel1_link">
-    <visual>
-        <origin rpy="1.570795 0 0" xyz="0 0 0"/>
-        <geometry><cylinder length="${d}" radius="${r}"/></geometry>
-    </visual>
-    <collision>
-        <origin rpy="1.570795 0 0" xyz="0 0 0"/>
-        <geometry><cylinder length="${d}" radius="${r}"/></geometry>
-    </collision>
-    <xacro:inertia_wheel />
-  </link>
-  <gazebo reference="${robot_name}/wheel1_link">
-    <mu1>1.0</mu1>
-    <mu2>1.0</mu2>
-    <kp>1000000.0</kp>
-    <kd>100.0</kd>
-    <minDepth>0.001</minDepth>
-    <maxVel>1.0</maxVel>
-  </gazebo>
-  <joint name="${robot_name}/wheel2_joint" type="continuous">
-    <parent link="${robot_name}/body_link"/>
-    <child link="${robot_name}/wheel2_link"/>
-    <origin xyz="${-s2} ${s4} ${-r}" rpy="0 0 0"/>
-    <axis xyz="0 1 0"/>
-    <limit effort="5000" velocity="10"/>
-    <dynamics damping="1.0" friction="1.0"/>
-  </joint>
-  <link name="${robot_name}/wheel2_link">
-    <visual>
-        <origin rpy="1.570795 0 0" xyz="0 0 0"/>
-        <geometry><cylinder length="${d}" radius="${r}"/></geometry>
-    </visual>
-    <collision>
-        <origin rpy="1.570795 0 0" xyz="0 0 0"/>
-        <geometry><cylinder length="${d}" radius="${r}"/></geometry>
-    </collision>
-    <xacro:inertia_wheel />
-  </link>
-  <gazebo reference="${robot_name}/wheel2_link">
-    <mu1>1.0</mu1>
-    <mu2>1.0</mu2>
-    <kp>1000000.0</kp>
-    <kd>100.0</kd>
-    <minDepth>0.001</minDepth>
-    <maxVel>1.0</maxVel>
-  </gazebo>
-  <joint name="${robot_name}/caster_joint" type="continuous">
-    <parent link="${robot_name}/body_link"/>
-    <child link="${robot_name}/caster_link"/>
-    <origin xyz="${s3} 0 ${-r}" rpy="0 0 0"/>
-    <axis xyz="0 1 0"/>
-  </joint>
-  <link name="${robot_name}/caster_link">
-    <visual>
-      <origin rpy="0 0 0" xyz="0 0 0"/>
-      <geometry><sphere radius="${r}"/></geometry>
-    </visual>
-    <collision>
-      <origin rpy="0 0 0" xyz="0 0 0"/>
-      <geometry><sphere radius="${r}"/></geometry>
-    </collision>
-    <xacro:inertia_caster />
-  </link>
-  <gazebo reference="${robot_name}/caster_link">
-    <mu1>0.0</mu1>
-    <mu2>0.0</mu2>
-    <material>Gazebo/Red</material>
-  </gazebo>
-  <joint name="${robot_name}/slope_joint" type="fixed">
-    <parent link="${robot_name}/body_link"/>
-    <child link="${robot_name}/slope_link"/>
-  </joint>
-  <link name="${robot_name}/slope_link">
-    <visual>
-      <origin xyz="${a/2} 0 ${-b/2}" rpy="3.14 2.54 0"/>
-      <geometry><box size="0.05 ${c} 0.25"/></geometry>
-    </visual>
-    <collision>
-      <geometry><box size="0.05 ${c} 0.25"/></geometry>
-      <origin xyz="${a/2} 0 ${b/2}" rpy="3.14 2.54 0"/>
-    </collision>
-  </link>
-  <gazebo reference="${robot_name}/slope_link">
-    <mu1>0.0</mu1>
-    <mu2>0.0</mu2>
-  </gazebo>
-  <joint name="${robot_name}/lidar_joint" type="fixed">
-    <origin xyz="0 0 0" rpy="0 0 0"/>
-    <parent link="${robot_name}/body_link"/>
-    <child link="${robot_name}/lidar_link"/>
-  </joint>
-  <link name="${robot_name}/lidar_link">
-    <visual>
-      <origin rpy="0 0 0.05" xyz="0.0 0 ${b/2 + 0.05}"/>
-      <geometry><cylinder length="0.1" radius="0.1"/></geometry>
-    </visual>
-    <collision>
-      <origin rpy="0 0 0" xyz="0.0 0 ${b/2 + 0.05}"/>
-      <geometry><cylinder length="0.1" radius="0.1"/></geometry>
-    </collision>
-    <inertial>
-      <mass value="0.01"/>
-      <origin rpy="0 0 0" xyz="0 0 0"/>
-      <inertia ixx="0.0001" ixy="0" ixz="0" iyy="0.0001" iyz="0" izz="0.0001"/>
-    </inertial>
-  </link>
-  <xacro:gazebo_config
-    robot_name="${robot_name}"
-    wheel1_joint="${robot_name}/wheel1_joint"
-    wheel2_joint="${robot_name}/wheel2_joint"
-    r="${r}"
-    s4="${s4}"
- />
-</xacro:macro>
-</robot>
+/home/adharsh/Desktop/Swarm-robot/build/mobile_robot/model/robot_macro.xacro

Commit message: corrected measurement and angle turning

File: install/mobile_robot/share/mobile_robot/model/robot1.xacro (robot description, xacro)
@@ -1 +1,5 @@
-/home/adharsh/Desktop/Swarm-robot/build/mobile_robot/model/robot1.xacro
+<?xml version="1.0"?>
+<robot name="differential_drive_robot" xmlns:xacro="http://www.ros.org/wiki/xacro">
+  <xacro:include filename="$(find mobile_robot)/model/robot_macro.xacro"/>
+  <xacro:differential_drive_robot robot_name="robot1"/>
+</robot>

File: install/mobile_robot/share/mobile_robot/model/robot2.xacro (robot description, xacro)
@@ -1 +1,5 @@
-/home/adharsh/Desktop/Swarm-robot/build/mobile_robot/model/robot2.xacro
+<?xml version="1.0"?>
+<robot name="differential_drive_robot" xmlns:xacro="http://www.ros.org/wiki/xacro">
+  <xacro:include filename="$(find mobile_robot)/model/robot_macro.xacro"/>
+  <xacro:differential_drive_robot robot_name="robot2"/>
+</robot>

File: install/mobile_robot/share/mobile_robot/model/robot_macro.xacro (robot description, xacro)
@@ -1 +1,188 @@
-/home/adharsh/Desktop/Swarm-robot/build/mobile_robot/model/robot_macro.xacro
+<?xml version="1.0"?>
+<robot xmlns:xacro="http://www.ros.org/wiki/xacro">
+<xacro:macro name="differential_drive_robot" params="robot_name">
+  <xacro:property name="pi_const" value="3.14159265"/>
+  <xacro:property name="r" value="0.15"/>
+  <xacro:property name="d" value="0.1"/>
+  <xacro:property name="a" value="1.0"/>
+  <xacro:property name="c" value="0.6"/>
+  <xacro:property name="b" value="0.3"/>
+  <xacro:property name="s1" value="${b/2+r}"/>
+  <xacro:property name="s2" value="${2*r}"/>
+  <xacro:property name="s3" value="${2*r}"/>
+  <xacro:property name="s4" value="${c/2+d/2+0.02}"/>
+  <xacro:property name="d1" value="200.0"/>
+  <xacro:property name="d2" value="500.0"/>
+  <xacro:property name="d3" value="200.0"/>
+  <xacro:property name="m1" value="${d1*a*b*c}"/>
+  <xacro:property name="m2" value="${d2*pi_const*r*r*d}"/>
+  <xacro:property name="m3" value="${d3*(4.0/3.0)*pi_const*r*r*r}"/>
+  <xacro:property name="Ix_body" value="${(1/12)*m1*(b*b+c*c)}"/>
+  <xacro:property name="Iy_body" value="${(1/12)*m1*(a*a+b*b)}"/>
+  <xacro:property name="Iz_body" value="${(1/12)*m1*(a*a+c*c)}"/>
+  <xacro:property name="Iz_wheel" value="${0.5*m2*r*r}"/>
+  <xacro:property name="I_wheel" value="${(1.0/12.0)*m2*(3.0*r*r+d*d)}"/>
+  <xacro:property name="I_caster" value="${(2.0/5.0)*m3*r*r}"/>
+  <xacro:macro name="inertia_body">
+    <inertial>
+      <origin rpy="0 0 0" xyz="0 0 0"/>
+      <mass value="${m1}"/>
+      <inertia ixx="${Ix_body}" ixy="0.0" ixz="0.0" iyy="${Iy_body}" iyz="0" izz="${Iz_body}" />
+    </inertial>
+  </xacro:macro>
+  <xacro:macro name="inertia_wheel">
+    <inertial>
+      <origin rpy="1.570795 0 0" xyz="0 0 0"/>
+      <mass value="${m2}"/>
+      <inertia ixx="${I_wheel}" ixy="0.0" ixz="0.0" iyy="${I_wheel}" iyz="0" izz="${Iz_wheel}" />
+    </inertial>
+  </xacro:macro>
+  <xacro:macro name="inertia_caster">
+    <inertial>
+      <origin rpy="0 0 0" xyz="0 0 0"/>
+      <mass value="${m3}"/>
+      <inertia ixx="${I_caster}" ixy="0.0" ixz="0.0" iyy="${I_caster}" iyz="0" izz="${I_caster}" />
+    </inertial>
+  </xacro:macro>
+  <xacro:include filename="$(find mobile_robot)/model/robot.gazebo"/>
+  <link name="${robot_name}/base_footprint"/>
+  <joint name="${robot_name}/body_link_joint" type="fixed">
+    <parent link="${robot_name}/base_footprint"/>
+    <child link="${robot_name}/body_link"/>
+    <origin xyz="0 0 ${2*r}" rpy="0 0 0"/>
+  </joint>
+  <link name="${robot_name}/body_link">
+    <visual>
+        <geometry><box size="${a} ${c} ${b}"/></geometry>
+        <origin rpy="0 0 0" xyz="0 0 0"/>
+    </visual>
+    <collision>
+        <geometry><box size="${a} ${c} ${b- 0.05}"/></geometry>
+        <origin rpy="0 0 0" xyz="0 0 0.025"/>
+    </collision>
+    <xacro:inertia_body />
+  </link>
+  <joint name="${robot_name}/wheel1_joint" type="continuous">
+    <parent link="${robot_name}/body_link"/>
+    <child link="${robot_name}/wheel1_link"/>
+    <origin xyz="${-s2} ${-s4} ${-r}" rpy="0 0 0"/>
+    <axis xyz="0 1 0"/>
+    <limit effort="5000" velocity="10"/>
+    <dynamics damping="1.0" friction="1.0"/>
+  </joint>
+  <link name="${robot_name}/wheel1_link">
+    <visual>
+        <origin rpy="1.570795 0 0" xyz="0 0 0"/>
+        <geometry><cylinder length="${d}" radius="${r}"/></geometry>
+    </visual>
+    <collision>
+        <origin rpy="1.570795 0 0" xyz="0 0 0"/>
+        <geometry><cylinder length="${d}" radius="${r}"/></geometry>
+    </collision>
+    <xacro:inertia_wheel />
+  </link>
+  <!-- <gazebo reference="${robot_name}/wheel1_link">
+    <mu1>1.0</mu1>
+    <mu2>1.0</mu2>
+    <kp>1000000.0</kp>
+    <kd>100.0</kd>
+    <minDepth>0.001</minDepth>
+    <maxVel>1.0</maxVel>
+  </gazebo> -->
+  <joint name="${robot_name}/wheel2_joint" type="continuous">
+    <parent link="${robot_name}/body_link"/>
+    <child link="${robot_name}/wheel2_link"/>
+    <origin xyz="${-s2} ${s4} ${-r}" rpy="0 0 0"/>
+    <axis xyz="0 1 0"/>
+    <limit effort="5000" velocity="10"/>
+    <dynamics damping="1.0" friction="1.0"/>
+  </joint>
+  <link name="${robot_name}/wheel2_link">
+    <visual>
+        <origin rpy="1.570795 0 0" xyz="0 0 0"/>
+        <geometry><cylinder length="${d}" radius="${r}"/></geometry>
+    </visual>
+    <collision>
+        <origin rpy="1.570795 0 0" xyz="0 0 0"/>
+        <geometry><cylinder length="${d}" radius="${r}"/></geometry>
+    </collision>
+    <xacro:inertia_wheel />
+  </link>
+  <!-- <gazebo reference="${robot_name}/wheel2_link">
+    <mu1>1.0</mu1>
+    <mu2>1.0</mu2>
+    <kp>1000000.0</kp>
+    <kd>100.0</kd>
+    <minDepth>0.001</minDepth>
+    <maxVel>1.0</maxVel>
+  </gazebo> -->
+  <joint name="${robot_name}/caster_joint" type="continuous">
+    <parent link="${robot_name}/body_link"/>
+    <child link="${robot_name}/caster_link"/>
+    <origin xyz="${s3} 0 ${-r}" rpy="0 0 0"/>
+    <axis xyz="0 1 0"/>
+  </joint>
+  <link name="${robot_name}/caster_link">
+    <visual>
+      <origin rpy="0 0 0" xyz="0 0 0"/>
+      <geometry><sphere radius="${r}"/></geometry>
+    </visual>
+    <collision>
+      <origin rpy="0 0 0" xyz="0 0 0"/>
+      <geometry><sphere radius="${r}"/></geometry>
+    </collision>
+    <xacro:inertia_caster />
+  </link>
+  <!-- <gazebo reference="${robot_name}/caster_link">
+    <mu1>0.0</mu1>
+    <mu2>0.0</mu2>
+    <material>Gazebo/Red</material>
+  </gazebo> -->
+  <joint name="${robot_name}/slope_joint" type="fixed">
+    <parent link="${robot_name}/body_link"/>
+    <child link="${robot_name}/slope_link"/>
+  </joint>
+  <link name="${robot_name}/slope_link">
+    <visual>
+      <origin xyz="${a/2} 0 ${-b/2}" rpy="3.14 2.54 0"/>
+      <geometry><box size="0.05 ${c} 0.25"/></geometry>
+    </visual>
+    <collision>
+      <geometry><box size="0.05 ${c} 0.25"/></geometry>
+      <origin xyz="${a/2} 0 ${b/2}" rpy="3.14 2.54 0"/>
+    </collision>
+  </link>
+  <!-- <gazebo reference="${robot_name}/slope_link">
+    <mu1>0.0</mu1>
+    <mu2>0.0</mu2>
+  </gazebo>
+   -->
+  <joint name="${robot_name}/lidar_joint" type="fixed">
+    <origin xyz="0 0 0" rpy="0 0 0"/>
+    <parent link="${robot_name}/body_link"/>
+    <child link="${robot_name}/lidar_link"/>
+  </joint>
+  <link name="${robot_name}/lidar_link">
+    <visual>
+      <origin rpy="0 0 0.05" xyz="0.0 0 ${b/2 + 0.05}"/>
+      <geometry><cylinder length="0.1" radius="0.1"/></geometry>
+    </visual>
+    <collision>
+      <origin rpy="0 0 0" xyz="0.0 0 ${b/2 + 0.05}"/>
+      <geometry><cylinder length="0.1" radius="0.1"/></geometry>
+    </collision>
+    <inertial>
+      <mass value="0.01"/>
+      <origin rpy="0 0 0" xyz="0 0 0"/>
+      <inertia ixx="0.0001" ixy="0" ixz="0" iyy="0.0001" iyz="0" izz="0.0001"/>
+    </inertial>
+  </link>
+  <xacro:gazebo_config
+    robot_name="${robot_name}"
+    wheel1_joint="${robot_name}/wheel1_joint"
+    wheel2_joint="${robot_name}/wheel2_joint"
+    r="${r}"
+    s4="${s4}"
+ />
+</xacro:macro>
+</robot>

File: src/mobile_robot/model/robot_macro.xacro (robot description, xacro)
@@ -11,8 +11,8 @@
   <xacro:property name="s2" value="${2*r}"/>
   <xacro:property name="s3" value="${2*r}"/>
-  <xacro:property name="s4" value="${c/2+d/2}"/>
-  <xacro:property name="d1" value="10.0"/>
-  <xacro:property name="d2" value="10.0"/>
-  <xacro:property name="d3" value="10.0"/>
+  <xacro:property name="s4" value="${c/2+d/2+0.02}"/>
+  <xacro:property name="d1" value="200.0"/>
+  <xacro:property name="d2" value="500.0"/>
+  <xacro:property name="d3" value="200.0"/>
   <xacro:property name="m1" value="${d1*a*b*c}"/>
   <xacro:property name="m2" value="${d2*pi_const*r*r*d}"/>
@@ -58,6 +58,6 @@
     </visual>
     <collision>
-        <geometry><box size="${a} ${c} ${b}"/></geometry>
-        <origin rpy="0 0 0" xyz="0 0 0"/>
+        <geometry><box size="${a} ${c} ${b- 0.05}"/></geometry>
+        <origin rpy="0 0 0" xyz="0 0 0.025"/>
     </collision>
     <xacro:inertia_body />
@@ -82,5 +82,5 @@
     <xacro:inertia_wheel />
   </link>
-  <gazebo reference="${robot_name}/wheel1_link">
+  <!-- <gazebo reference="${robot_name}/wheel1_link">
     <mu1>1.0</mu1>
     <mu2>1.0</mu2>
@@ -89,5 +89,5 @@
     <minDepth>0.001</minDepth>
     <maxVel>1.0</maxVel>
-  </gazebo>
+  </gazebo> -->
   <joint name="${robot_name}/wheel2_joint" type="continuous">
     <parent link="${robot_name}/body_link"/>
@@ -109,5 +109,5 @@
     <xacro:inertia_wheel />
   </link>
-  <gazebo reference="${robot_name}/wheel2_link">
+  <!-- <gazebo reference="${robot_name}/wheel2_link">
     <mu1>1.0</mu1>
     <mu2>1.0</mu2>
@@ -116,5 +116,5 @@
     <minDepth>0.001</minDepth>
     <maxVel>1.0</maxVel>
-  </gazebo>
+  </gazebo> -->
   <joint name="${robot_name}/caster_joint" type="continuous">
     <parent link="${robot_name}/body_link"/>
@@ -134,9 +134,9 @@
     <xacro:inertia_caster />
   </link>
-  <gazebo reference="${robot_name}/caster_link">
+  <!-- <gazebo reference="${robot_name}/caster_link">
     <mu1>0.0</mu1>
     <mu2>0.0</mu2>
     <material>Gazebo/Red</material>
-  </gazebo>
+  </gazebo> -->
   <joint name="${robot_name}/slope_joint" type="fixed">
     <parent link="${robot_name}/body_link"/>
@@ -153,8 +153,9 @@
     </collision>
   </link>
-  <gazebo reference="${robot_name}/slope_link">
+  <!-- <gazebo reference="${robot_name}/slope_link">
     <mu1>0.0</mu1>
     <mu2>0.0</mu2>
   </gazebo>
+   -->
   <joint name="${robot_name}/lidar_joint" type="fixed">
     <origin xyz="0 0 0" rpy="0 0 0"/>
